File: Hardware/Rev.C/Amaranth/Amaranth.kicad_pcb (KiCad board)
At the start: 4 copper layers, 150 x 118 mm, 81 parts, among them J1 RJ45_LED, J2 IDE, J3 ATX24, J4 KBD, J5 VGA, P1 JTAG, SW1 SW_SPDT, U1 MCF5208, U10 IS61WV25616, U12 10M04SCE144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

Commit message: updated schematic
Parts:
- added U6: 74LVC16245A, Package_SO:TSSOP-48_6.1x12.5mm_P0.5mm, F.Cu at (47.8, 78.2)
- added U7: 74LVC16245A, Package_SO:TSSOP-48_6.1x12.5mm_P0.5mm, F.Cu at (61.8, 78.2)
- moved U9 144.1 mm to (163.0, 181.5)
- moved U10 123.1 mm to (149.2, 181.5)
- moved R1 59.5 mm to (50.5, 175.8), turned to 90 degrees
- moved U1 41.1 mm to (69.2, 180.0)
- moved U4 26.3 mm to (135.5, 181.5)
- moved U5 13.0 mm to (121.2, 181.5)
- moved U2 11.7 mm to (99.2, 179.8)
- moved U3 4.89 mm to (108.8, 179.8)
Routing:
- net GND: track 213.9 -> 342.4 mm, vias 170 -> 142
- net Net-(U7-Pad11): track 0.00 -> 69.0 mm, vias 0 -> 2
- net /DL23: track 69.0 -> 0.00 mm, vias 2 -> 0
- net +3V3: track 55.8 -> 124.1 mm, vias 30 -> 16
- net Net-(U7-Pad8): track 0.00 -> 47.3 mm, vias 0 -> 2
- net /DL21: track 47.3 -> 0.00 mm, vias 2 -> 0
- net /DL22: track 46.8 -> 0.00 mm, vias 2 -> 0
- net /DL20: track 45.6 -> 0.00 mm, vias 2 -> 0
- net /DL7: track 114.9 -> 73.3 mm, vias 7 -> 3
- net Net-(U7-Pad2): track 0.00 -> 40.4 mm, vias 0 -> 2
- net /DL17: track 40.4 -> 0.00 mm, vias 2 -> 0
- net /DL4: track 97.8 -> 58.2 mm, vias 8 -> 4
- net Net-(U7-Pad5): track 0.00 -> 39.5 mm, vias 0 -> 2
- net /DL19: track 39.5 -> 0.00 mm, vias 2 -> 0
- net /DL18: track 38.9 -> 0.00 mm, vias 2 -> 0
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
Commit message: Routed a bit of the new SRAM stuff
Parts:
- moved U18 169.8 mm to (59.0, 225.6)
- moved U6 158.3 mm to (73.0, 234.6), turned to 0 degrees
- moved RN1 153.5 mm to (120.0, 218.1)
- moved U7 143.2 mm to (73.0, 221.1), turned to 0 degrees
- moved U4 56.1 mm to (171.0, 225.0)
- moved U1 49.7 mm to (94.2, 223.0)
- moved U9 47.9 mm to (143.0, 225.0)
- moved U10 44.2 mm to (157.0, 225.0)
- moved U5 44.2 mm to (129.0, 225.0)
Connections:
- net 8b_L5 renamed Net-(U12-Pad57)
- net 8b_L6 renamed Net-(U12-Pad58)
- net 8b_L7 renamed Net-(U12-Pad59)
- net CS_FLOPPY renamed Net-(U12-Pad140)
- net CS_FLOPPY_LDCR renamed Net-(U12-Pad138)
- U12 pad 12: 8burst_2 -> Net-(U12-Pad12)
- U12 pad 13: 8burst_3 -> Net-(U12-Pad13)
- U12 pad 136: CS_FLOPPY_LDOR -> CS_ROM
- U12 pad 141: CS_ROM -> Net-(U12-Pad141)
- U12 pad 56: 8b_L4 -> 8b_OUT
- U12 pad 60: 8b_OUT -> Net-(U12-Pad60)
- U18 pad 10: 8burst_2 -> /A2
- U18 pad 13: /DL0 -> /DR0
- U18 pad 14: /DL1 -> /DR1
- U18 pad 15: /DL2 -> /DR2
- U18 pad 17: /DL3 -> /DR3
- U18 pad 18: /DL4 -> /DR4
- U18 pad 19: /DL5 -> /DR5
- U18 pad 20: /DL6 -> /DR6
- U18 pad 21: /DL7 -> /DR7
- U18 pad 9: 8burst_3 -> /A3
- U6 pad 1: Net-(U6-Pad1) -> 8b_OUT
- U6 pad 11: Net-(U6-Pad11) -> /DR6
- U6 pad 12: Net-(U6-Pad12) -> /DR7
- U6 pad 13: Net-(U6-Pad13) -> /DR0
- U6 pad 14: Net-(U6-Pad14) -> /DR1
- U6 pad 16: Net-(U6-Pad16) -> /DR2
- U6 pad 17: Net-(U6-Pad17) -> /DR3
- U6 pad 19: Net-(U6-Pad19) -> /DR4
- U6 pad 2: Net-(U6-Pad2) -> /DR0
- U6 pad 20: Net-(U6-Pad20) -> /DR5
- U6 pad 22: Net-(U6-Pad22) -> /DR6
- U6 pad 23: Net-(U6-Pad23) -> /DR7
- U6 pad 24: Net-(U6-Pad24) -> 8b_OUT
- U6 pad 25: Net-(U6-Pad25) -> 8b_L1
- U6 pad 26: Net-(U6-Pad26) -> /DL15
- U6 pad 27: Net-(U6-Pad27) -> /DL14
- U6 pad 29: Net-(U6-Pad29) -> /DL13
- U6 pad 3: Net-(U6-Pad3) -> /DR1
- U6 pad 30: Net-(U6-Pad30) -> /DL12
- U6 pad 32: Net-(U6-Pad32) -> /DL11
- U6 pad 33: Net-(U6-Pad33) -> /DL10
- U6 pad 35: Net-(U6-Pad35) -> /DL9
- U6 pad 36: Net-(U6-Pad36) -> /DL8
- U6 pad 37: Net-(U6-Pad37) -> /DL7
- U6 pad 38: Net-(U6-Pad38) -> /DL6
- U6 pad 40: Net-(U6-Pad40) -> /DL5
- U6 pad 41: Net-(U6-Pad41) -> /DL4
- U6 pad 43: Net-(U6-Pad43) -> /DL3
- U6 pad 44: Net-(U6-Pad44) -> /DL2
- U6 pad 46: Net-(U6-Pad46) -> /DL1
- U6 pad 47: Net-(U6-Pad47) -> /DL0
- U6 pad 48: Net-(U6-Pad48) -> 8b_L0
- U6 pad 5: Net-(U6-Pad5) -> /DR2
- U6 pad 6: Net-(U6-Pad6) -> /DR3
- U6 pad 8: Net-(U6-Pad8) -> /DR4
- U6 pad 9: Net-(U6-Pad9) -> /DR5
- U7 pad 1: Net-(U7-Pad1) -> 8b_OUT
- U7 pad 11: Net-(U7-Pad11) -> /DR6
- U7 pad 12: Net-(U7-Pad12) -> /DR7
- U7 pad 13: Net-(U7-Pad13) -> /DR0
- U7 pad 14: Net-(U7-Pad14) -> /DR1
- U7 pad 16: Net-(U7-Pad16) -> /DR2
- U7 pad 17: Net-(U7-Pad17) -> /DR3
- U7 pad 19: Net-(U7-Pad19) -> /DR4
- U7 pad 2: Net-(U7-Pad2) -> /DR0
- U7 pad 20: Net-(U7-Pad20) -> /DR5
- U7 pad 22: Net-(U7-Pad22) -> /DR6
- U7 pad 23: Net-(U7-Pad23) -> /DR7
- U7 pad 24: Net-(U7-Pad24) -> 8b_OUT
- U7 pad 25: Net-(U7-Pad25) -> 8b_L3
- U7 pad 26: Net-(U7-Pad26) -> /DL31
- U7 pad 27: Net-(U7-Pad27) -> /DL30
- U7 pad 29: Net-(U7-Pad29) -> /DL29
- U7 pad 3: Net-(U7-Pad3) -> /DR1
- U7 pad 30: Net-(U7-Pad30) -> /DL28
- U7 pad 32: Net-(U7-Pad32) -> /DL27
- U7 pad 33: Net-(U7-Pad33) -> /DL26
- U7 pad 35: Net-(U7-Pad35) -> /DL25
- U7 pad 36: Net-(U7-Pad36) -> /DL24
- U7 pad 37: Net-(U7-Pad37) -> /DL23
- U7 pad 38: Net-(U7-Pad38) -> /DL22
- U7 pad 40: Net-(U7-Pad40) -> /DL21
- U7 pad 41: Net-(U7-Pad41) -> /DL20
- U7 pad 43: Net-(U7-Pad43) -> /DL19
- U7 pad 44: Net-(U7-Pad44) -> /DL18
- U7 pad 46: Net-(U7-Pad46) -> /DL17
- U7 pad 47: Net-(U7-Pad47) -> /DL16
- U7 pad 48: Net-(U7-Pad48) -> 8b_L2
- U7 pad 5: Net-(U7-Pad5) -> /DR2
- U7 pad 6: Net-(U7-Pad6) -> /DR3
- U7 pad 8: Net-(U7-Pad8) -> /DR4
- U7 pad 9: Net-(U7-Pad9) -> /DR5
Routing:
- net /DR6: track 0.00 -> 180.7 mm, vias 0 -> 6
- net /DR0: track 0.00 -> 156.4 mm, vias 0 -> 7
- net /DR2: track 0.00 -> 156.3 mm, vias 0 -> 7
- net /DR4: track 0.00 -> 136.1 mm, vias 0 -> 7
- net /DR7: track 0.00 -> 112.7 mm, vias 0 -> 4
- net /DR5: track 0.00 -> 78.8 mm, vias 0 -> 8
- net /DR3: track 0.00 -> 71.5 mm, vias 0 -> 8
- net Net-(U7-Pad11): track 69.0 -> 0.00 mm, vias 2 -> 0
- net /DR1: track 0.00 -> 68.0 mm, vias 0 -> 8
- net /DL7: track 73.3 -> 17.4 mm, vias 3 -> 2
- net /DL5: track 74.0 -> 18.7 mm, vias 4 -> 3
- net /A14: track 171.8 -> 224.9 mm, vias 4 -> 8
- net /A16: track 176.5 -> 229.4 mm, vias 5 -> 9
- net /A12: track 176.1 -> 229.0 mm, vias 4 -> 8
- net /A9: track 116.5 -> 168.2 mm, vias 2 -> 6
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Other:
- net class Default: trace_width 0.25 -> 0.2; via_dia 0.8 -> 0.6; via_drill 0.4 -> 0.35
