File: Hardware/Rev.C/Amaranth/Amaranth.sch (KiCad schematic (older format))
At the start: 81 parts, among them J1 RJ45_LED, J2 IDE, J3 ATX24, J4 KBD, J5 VGA, P1 JTAG, SW1 SW_SPDT, U1 MCF5208, U10 IS61WV25616, U12 10M04SCE144, U13 ENC624J600-I_PT, U14 10M04SCE144, U18 SST39SF040, U2 AS4C16M16SA, U20 74LVC16245A, U3 AS4C16M16SA, U4 IS61WV25616, U5 IS61WV25616, U9 IS61WV25616, Y1 25MHz, Y2 100MHz

Commit message: updated schematic
Parts:
- added U6, U7: 74LVC16245A, Package_SO:TSSOP-48_6.1x12.5mm_P0.5mm, symbol Amaranth:74LVC16373A
Connections:
- net +3V3: now also U6.18 (VCC-2), U6.31 (VCC-3), U6.42 (VCC), U6.7 (VCC-1), U7.18 (VCC-2), U7.31 (VCC-3), U7.42 (VCC), U7.7 (VCC-1)
- net GND: now also U6.10 (GND-4), U6.15 (GND-5), U6.21 (GND), U6.28 (GND-1), U6.34 (GND-7), U6.39 (GND-6), U6.4 (GND-3), U6.45 (GND-2), U7.10 (GND-4), U7.15 (GND-5), U7.21 (GND), U7.28 (GND-1), U7.34 (GND-7), U7.39 (GND-6), U7.4 (GND-3), U7.45 (GND-2)
Changed lines of the file:
@@
 	34900 1000 33000 1000
 Connection ~ 29500 1000
+Connection ~ 33000 1000
+Wire Bus Line
+	33000 1000 29500 1000
+$Comp
+L power:GND #PWR0122
+U 1 1 5D6F2217
+P 10000 7700
+F 0 "#PWR0122" H 10000 7450 50  0001 C CNN
+F 1 "GND" H 10005 7527 50  0000 C CNN
+F 2 "" H 10000 7700 50  0001 C CNN
+F 3 "" H 10000 7700 50  0001 C CNN
+	1    10000 7700
+	-1   0    0    -1
+$EndComp
+$Comp
+L Amaranth:74LVC16373A U6
+U 1 1 5D6F221D
+P 10000 6800
+F 0 "U6" H 9700 8050 50  0000 C CNN
+F 1 "74LVC16245A" H 10350 5850 50  0000 C CNN
+F 2 "Package_SO:TSSOP-48_6.1x12.5mm_P0.5mm" H 10700 8450 50  0001 C CNN
+F 3 "" H 10700 8450 50  0001 C CNN
+	1    10000 6800
+	1    0    0    -1
+$EndComp
+$Comp
+L power:+3V3 #PWR0123
+U 1 1 5D6F2223
+P 10000 5600
+F 0 "#PWR0123" H 10000 5450 50  0001 C CNN
+F 1 "+3V3" H 10015 5773 50  0000 C CNN
+F 2 "" H 10000 5600 50  0001 C CNN
+F 3 "" H 10000 5600 50  0001 C CNN
+	1    10000 5600
+	1    0    0    -1
+$EndComp
+$Comp
+L power:GND #PWR0124
+U 1 1 5D8C7CC5
+P 10000 10300
+F 0 "#PWR0124" H 10000 10050 50  0001 C CNN
+F 1 "GND" H 10005 10127 50  0000 C CNN
+F 2 "" H 10000 10300 50  0001 C CNN
+F 3 "" H 10000 10300 50  0001 C CNN
+	1    10000 10300
+	-1   0    0    -1
+$EndComp
+$Comp
+L Amaranth:74LVC16373A U7
+U 1 1 5D8C7CCB
+P 10000 9400
+F 0 "U7" H 9700 10650 50  0000 C CNN
+F 1 "74LVC16245A" H 10350 8450 50  0000 C CNN
+F 2 "Package_SO:TSSOP-48_6.1x12.5mm_P0.5mm" H 10700 11050 50  0001 C CNN
+F 3 "" H 10700 11050 50  0001 C CNN
+	1    10000 9400
+	1    0    0    -1
+$EndComp
+$Comp
+L power:+3V3 #PWR0125
+U 1 1 5D8C7CD1
+P 10000 8200
+F 0 "#PWR0125" H 10000 8050 50  0001 C CNN
+F 1 "+3V3" H 10015 8373 50  0000 C CNN
+F 2 "" H 10000 8200 50  0001 C CNN
+F 3 "" H 10000 8200 50  0001 C CNN
+	1    10000 8200
+	1    0    0    -1
+$EndComp
 Wire Bus Line
 	9000 1200 9000 2400
+Wire Bus Line
+	27400 1200 27400 4050
 Wire Bus Line
 	2800 20550 2800 21650
@@
 Wire Bus Line
 	19300 15100 19300 16650
-Wire Bus Line
-	27400 1200 27400 4050
 Wire Bus Line
 	10800 1000 10800 3500
@@
 Wire Bus Line
 	6600 1300 6600 4800
-Connection ~ 33000 1000
-Wire Bus Line
-	33000 1000 29500 1000
 $EndSCHEMATC

Commit message: Routed a bit of the new SRAM stuff
Connections:
- net 8b_L4 is gone; now on net 8b_OUT: U12.56 (IO3/DIFFIO_TX_RX_B12p/DIFFOUT_B12p)
- net CS_FLOPPY_LDOR is gone; now on net CS_ROM: U12.136 (IO8/DIFFIO_RX_T24p/DIFFOUT_T24p/nSTATUS)
- net 8b_L0: now also U6.48 (1LE)
- net 8b_L1: now also U6.25 (2LE)
- net 8b_L2: now also U7.48 (1LE)
- net 8b_L3: now also U7.25 (2LE)
- net 8b_OUT: now also U6.1 (~1OE), U6.24 (~2OE), U7.1 (~1OE), U7.24 (~2OE); no longer U12.60 (IO3/DIFFIO_TX_RX_B16p/DIFFOUT_B16p)
- net A2: now also U18.10 (A2)
- net A3: now also U18.9 (A3)
- net CS_ROM: no longer U12.141 (IO8/DIFFIO_RX_T26n/DIFFOUT_T26n)
- net DL0: now also U6.47 (1D1); no longer U18.13 (D0)
- net DL1: now also U6.46 (1D2); no longer U18.14 (D1)
- net DL10: now also U6.33 (2D3)
- net DL11: now also U6.32 (2D4)
- net DL12: now also U6.30 (2D5)
- net DL13: now also U6.29 (2D6)
- net DL14: now also U6.27 (2D7)
- net DL15: now also U6.26 (2D8)
- net DL16: now also U7.47 (1D1)
- net DL17: now also U7.46 (1D2)
- net DL18: now also U7.44 (1D3)
- net DL19: now also U7.43 (1D4)
- net DL2: now also U6.44 (1D3); no longer U18.15 (D2)
- net DL20: now also U7.41 (1D5)
- net DL21: now also U7.40 (1D6)
- net DL22: now also U7.38 (1D7)
- net DL23: now also U7.37 (1D8)
- net DL24: now also U7.36 (2D1)
- net DL25: now also U7.35 (2D2)
- net DL26: now also U7.33 (2D3)
- net DL27: now also U7.32 (2D4)
- net DL28: now also U7.30 (2D5)
- net DL29: now also U7.29 (2D6)
- net DL3: now also U6.43 (1D4); no longer U18.17 (D3)
- net DL30: now also U7.27 (2D7)
- net DL31: now also U7.26 (2D8)
- net DL4: now also U6.41 (1D5); no longer U18.18 (D4)
- net DL5: now also U6.40 (1D6); no longer U18.19 (D5)
- net DL6: now also U6.38 (1D7); no longer U18.20 (D6)
- net DL7: now also U6.37 (1D8); no longer U18.21 (D7)
- net DL8: now also U6.36 (2D1)
- net DL9: now also U6.35 (2D2)
- net DR6: now reaches U6.11 (1Q7)
- net DR6: now also U18.20 (D6), U6.22 (2Q7), U7.11 (1Q7), U7.22 (2Q7)
- net DR7: now reaches U6.12 (1Q8)
- net DR7: now also U18.21 (D7), U6.23 (2Q8), U7.12 (1Q8), U7.23 (2Q8)
- net DR0: now reaches U6.13 (2Q1)
- net DR0: now also U18.13 (D0), U6.2 (1Q1), U7.13 (2Q1), U7.2 (1Q1)
- net DR1: now reaches U6.14 (2Q2)
- net DR1: now also U18.14 (D1), U6.3 (1Q2), U7.14 (2Q2), U7.3 (1Q2)
- net DR2: now reaches U6.16 (2Q3)
- net DR2: now also U18.15 (D2), U6.5 (1Q3), U7.16 (2Q3), U7.5 (1Q3)
- net DR3: now reaches U6.17 (2Q4)
- net DR3: now also U18.17 (D3), U6.6 (1Q4), U7.17 (2Q4), U7.6 (1Q4)
- net DR4: now reaches U6.19 (2Q5)
- net DR4: now also U18.18 (D4), U6.8 (1Q5), U7.19 (2Q5), U7.8 (1Q5)
- net DR5: now reaches U6.20 (2Q6)
- net DR5: now also U18.19 (D5), U6.9 (1Q6), U7.20 (2Q6), U7.9 (1Q6)
- net 8b_L5: no longer names the net of U12.57 (IO3/DIFFIO_TX_RX_B14n/DIFFOUT_B14n)
- net 8b_L6: no longer names the net of U12.58 (IO3/DIFFIO_TX_RX_B14p/DIFFOUT_B14p)
- net 8b_L7: no longer names the net of U12.59 (IO3/DIFFIO_TX_RX_B16n/DIFFOUT_B16n)
- net 8burst_2: no longer names the net of U12.12 (IO1A/DIFFIO_RX_L5p/DIFFOUT_L5p)
- net 8burst_2: no longer U18.10 (A2)
- net 8burst_3: no longer names the net of U12.13 (IO1A/DIFFIO_RX_L7n/DIFFOUT_L7n)
- net 8burst_3: no longer U18.9 (A3)
- net CS_FLOPPY: no longer names the net of U12.140 (IO8/DIFFIO_RX_T26p/DIFFOUT_T26p)
- net CS_FLOPPY_LDCR: no longer names the net of U12.138 (IO8/DIFFIO_RX_T24n/DIFFOUT_T24n/CONF_DONE)
Other:
- moved on the sheet: J4, R11, R12, R13, R14, U12A, U12B, U12C, U18, U6, U7
